Commit message: Fix + Pipe and Robot STL Integration

File: practice_agos/agos_sim/urdf/agos_materials.xacro (robot description, xacro)
@@ -1,25 +1,23 @@
 <?xml version="1.0"?>
 <robot xmlns:xacro="http://www.ros.org/wiki/xacro">
-  <material name="agos_chassis_grey">
-    <color rgba="0.35 0.35 0.38 1.0"/>
+  <!-- Colours of the CAD parts (read from the per-face colours stored in
+       Designs/STL/AGOS V1.stl) -->
+  <material name="agos_body_grey">
+    <color rgba="0.62 0.62 0.63 1.0"/>
   </material>
-  <material name="agos_track_black">
+  <material name="agos_tread_red">
+    <color rgba="0.74 0.19 0.13 1.0"/>
+  </material>
+  <material name="agos_accent_yellow">
+    <color rgba="0.90 0.68 0.13 1.0"/>
+  </material>
+  <material name="agos_light_grey">
+    <color rgba="0.94 0.94 0.93 1.0"/>
+  </material>
+  <material name="agos_green_body">
+    <color rgba="0.26 0.58 0.26 1.0"/>
+  </material>
+  <material name="agos_sensor_dark">
     <color rgba="0.08 0.08 0.08 1.0"/>
   </material>
-  <material name="agos_sensor_dark">
-    <color rgba="0.10 0.10 0.12 1.0"/>
-  </material>
-  <!-- Added from the primitive-shape design -->
-  <material name="agos_green_body">
-    <color rgba="0.15 0.55 0.25 1.0"/>
-  </material>
-  <material name="agos_silver_enclosure">
-    <color rgba="0.75 0.75 0.78 1.0"/>
-  </material>
-  <material name="agos_dark_grey_frame">
-    <color rgba="0.20 0.20 0.20 1.0"/>
-  </material>
-  <material name="agos_lidar_yellow">
-    <color rgba="0.95 0.70 0.00 1.0"/>
-  </material>
 </robot>

File: practice_agos/agos_sim/urdf/agos_sensors.xacro (robot description, xacro)
@@ -1,15 +1,10 @@
 <?xml version="1.0"?>
 <robot xmlns:xacro="http://www.ros.org/wiki/xacro">
+  <!-- Sensor positions are taken from Designs/STL/AGOS V1.stl. The sensors'
+       shapes are already part of the chassis mesh, so these links only carry
+       frames, a small mass and the Gazebo sensor definitions. -->
   <!-- ===================== Orbbec front-facing RGB-D camera ===================== -->
   <xacro:macro name="agos_camera">
-    <xacro:property name="cam_size" value="0.045"/>
     <link name="camera_link">
-      <visual>
-        <geometry><box size="${cam_size} 0.09 ${cam_size}"/></geometry>
-        <material name="agos_sensor_dark"/>
-      </visual>
-      <collision>
-        <geometry><box size="${cam_size} 0.09 ${cam_size}"/></geometry>
-      </collision>
       <inertial>
         <mass value="0.12"/>
@@ -18,8 +13,9 @@
       </inertial>
     </link>
+    <!-- Centre of the lens panel on the CAD camera, on top of the front of the lid -->
     <joint name="camera_joint" type="fixed">
       <parent link="chassis_link"/>
       <child link="camera_link"/>
-      <origin xyz="${chassis_length/2 + cam_size/2} 0 ${chassis_height*0.25}" rpy="0 0 0"/>
+      <origin xyz="0.331 0 0.2465" rpy="0 0 0"/>
     </joint>
     <!-- Optical frame: images/pointclouds must be stamped z-forward/x-right/y-down -->
@@ -30,6 +26,11 @@
       <origin xyz="0 0 0" rpy="${-pi/2} 0 ${-pi/2}"/>
     </joint>
+    <!-- Keep camera_link as its own link in Gazebo so the headlight below
+         stays at the camera instead of being merged into the chassis. -->
+    <gazebo reference="camera_joint">
+      <preserveFixedJoint>true</preserveFixedJoint>
+    </gazebo>
     <!-- Publishes (after ros_gz_bridge remap in config/bridge.yaml):
-         /camera/image_raw and /camera/depth/points -->
+         /camera/image_raw, /camera/depth/image_raw, /camera/depth/points -->
     <gazebo reference="camera_link">
       <sensor name="orbbec_rgbd_camera" type="rgbd_camera">
@@ -52,29 +53,41 @@
         </camera>
       </sensor>
+      <!-- Front LED headlight (the proposal's high-intensity front LED).
+           Without it the inside of the pipe is lit by ambient light only. -->
+      <light name="agos_headlight" type="spot">
+        <pose>0.03 0 0 0 0 0</pose>
+        <direction>1 0 0</direction>
+        <diffuse>1.0 0.97 0.9 1</diffuse>
+        <specular>0.3 0.3 0.3 1</specular>
+        <attenuation>
+          <range>6.0</range>
+          <constant>0.4</constant>
+          <linear>0.1</linear>
+          <quadratic>0.02</quadratic>
+        </attenuation>
+        <spot>
+          <inner_angle>0.5</inner_angle>
+          <outer_angle>1.1</outer_angle>
+          <falloff>1.0</falloff>
+        </spot>
+        <cast_shadows>false</cast_shadows>
+      </light>
     </gazebo>
   </xacro:macro>
-  <!-- ===================== Okdo 2D LiDAR ===================== -->
+  <!-- ===================== Okdo LD06 2D LiDAR ===================== -->
   <xacro:macro name="agos_lidar">
-    <xacro:property name="lidar_radius" value="0.035"/>
-    <xacro:property name="lidar_height" value="0.04"/>
     <link name="lidar_link">
-      <visual>
-        <geometry><cylinder radius="${lidar_radius}" length="${lidar_height}"/></geometry>
-        <material name="agos_sensor_dark"/>
-      </visual>
-      <collision>
-        <geometry><cylinder radius="${lidar_radius}" length="${lidar_height}"/></geometry>
-      </collision>
       <inertial>
-        <mass value="0.15"/>
+        <mass value="0.05"/>
         <origin xyz="0 0 0" rpy="0 0 0"/>
-        <inertia ixx="0.0001" ixy="0.0" ixz="0.0" iyy="0.0001" iyz="0.0" izz="0.0001"/>
+        <inertia ixx="0.00001" ixy="0.0" ixz="0.0" iyy="0.00001" iyz="0.0" izz="0.00001"/>
       </inertial>
     </link>
-    <!-- Sits on the yellow pedestal defined in agos.urdf.xacro (lidar_mount_h) -->
+    <!-- Scan plane of the LD06 on top of the lid (CAD LiDAR body: z 0.265-0.298).
+         It sits 1 cm above the top of the camera, so the camera does not block it. -->
     <joint name="lidar_joint" type="fixed">
       <parent link="chassis_link"/>
       <child link="lidar_link"/>
-      <origin xyz="0 0 ${chassis_height/2 + lidar_mount_h + lidar_height/2}" rpy="0 0 0"/>
+      <origin xyz="0 0 0.287" rpy="0 0 0"/>
     </joint>
     <gazebo reference="lidar_link">
@@ -104,11 +117,4 @@
   <xacro:macro name="agos_imu">
     <link name="imu_link">
-      <visual>
-        <geometry><box size="0.03 0.03 0.01"/></geometry>
-        <material name="agos_sensor_dark"/>
-      </visual>
-      <collision>
-        <geometry><box size="0.03 0.03 0.01"/></geometry>
-      </collision>
       <inertial>
         <mass value="0.05"/>
@@ -117,4 +123,5 @@
       </inertial>
     </link>
+    <!-- Inside the body, at the CAD origin -->
     <joint name="imu_joint" type="fixed">
       <parent link="chassis_link"/>
@@ -122,6 +129,6 @@
       <origin xyz="0 0 0.01" rpy="0 0 0"/>
     </joint>
-    <!-- Requires the gz-sim-imu-system world plugin (added in worlds/pvc_pipe.sdf)
-         or this topic stays silent even though the sensor is declared here. -->
+    <!-- Requires the gz-sim-imu-system world plugin (in worlds/agos_pipe.sdf
+         and worlds/agos_world.sdf) or this topic stays silent. -->
     <gazebo reference="imu_link">
       <sensor name="agos_imu" type="imu">

File: practice_agos/agos_sim/urdf/agos_tracks.xacro (robot description, xacro)
@@ -1,18 +1,16 @@
 <?xml version="1.0"?>
 <robot xmlns:xacro="http://www.ros.org/wiki/xacro">
-  <!-- Added 'mu' parameter to control friction per-wheel -->
-  <xacro:macro name="agos_wheel" params="side y_sign pos x mu">
+  <!-- Each track is modelled as driven wheel cylinders where the real track
+       touches things (cheap and stable). They have no visual: the track you
+       see is the CAD mesh on chassis_link.
+         4 road wheels  : the CAD rollers, bottoms on the ground (z = 0)
+         2 idler wheels : the raised front/rear ends of the track, so the
+                          robot can climb onto lips, debris and pipe walls -->
+  <xacro:macro name="agos_wheel" params="side y_sign pos x z mu">
     <link name="${side}_wheel_${pos}">
-      <visual>
-        <origin xyz="0 0 0" rpy="${pi/2} 0 0"/>
-        <geometry>
-          <cylinder radius="${track_radius - 0.012}" length="${track_width - 0.01}"/>
-        </geometry>
-        <material name="agos_track_black"/>
-      </visual>
       <collision>
         <origin xyz="0 0 0" rpy="${pi/2} 0 0"/>
         <geometry>
-          <cylinder radius="${track_radius}" length="${track_width - 0.01}"/>
+          <cylinder radius="${wheel_radius}" length="${track_width}"/>
         </geometry>
       </collision>
@@ -21,7 +19,7 @@
         <origin xyz="0 0 0" rpy="0 0 0"/>
         <inertia
-          ixx="${(wheel_mass/12.0)*(3*track_radius*track_radius + track_width*track_width)}" ixy="0.0" ixz="0.0"
-          iyy="${(wheel_mass/2.0)*track_radius*track_radius}" iyz="0.0"
-          izz="${(wheel_mass/12.0)*(3*track_radius*track_radius + track_width*track_width)}"/>
+          ixx="${(wheel_mass/12.0)*(3*wheel_radius*wheel_radius + track_width*track_width)}" ixy="0.0" ixz="0.0"
+          iyy="${(wheel_mass/2.0)*wheel_radius*wheel_radius}" iyz="0.0"
+          izz="${(wheel_mass/12.0)*(3*wheel_radius*wheel_radius + track_width*track_width)}"/>
       </inertial>
     </link>
@@ -29,10 +27,9 @@
       <parent link="base_link"/>
       <child link="${side}_wheel_${pos}"/>
-      <origin xyz="${x} ${y_sign * track_separation/2} 0" rpy="0 0 0"/>
+      <origin xyz="${x} ${y_sign * track_y} ${z}" rpy="0 0 0"/>
       <axis xyz="0 1 0"/>
       <dynamics damping="0.1" friction="0.05"/>
     </joint>
     <gazebo reference="${side}_wheel_${pos}">
-      <!-- Apply the specific friction passed into the macro -->
       <mu1>${mu}</mu1>
       <mu2>${mu}</mu2>
@@ -40,51 +37,30 @@
   </xacro:macro>
   <xacro:macro name="agos_track" params="side y_sign">
-    <link name="${side}_track_frame">
-      <!-- center straight section -->
-      <visual>
-        <origin xyz="0 0 0" rpy="0 0 0"/>
-        <geometry>
-          <box size="${2*wheel_x_offset} ${track_width} ${2*track_radius}"/>
-        </geometry>
-        <material name="agos_track_black"/>
-      </visual>
-      <!-- front rounded end -->
-      <visual>
-        <origin xyz="${wheel_x_offset} 0 0" rpy="${pi/2} 0 0"/>
-        <geometry>
-          <cylinder radius="${track_radius}" length="${track_width}"/>
-        </geometry>
-        <material name="agos_track_black"/>
-      </visual>
-      <!-- rear rounded end -->
-      <visual>
-        <origin xyz="${-wheel_x_offset} 0 0" rpy="${pi/2} 0 0"/>
-        <geometry>
-          <cylinder radius="${track_radius}" length="${track_width}"/>
-        </geometry>
-        <material name="agos_track_black"/>
-      </visual>
-    </link>
-    <joint name="${side}_track_frame_joint" type="fixed">
-      <parent link="base_link"/>
-      <child link="${side}_track_frame"/>
-      <origin xyz="0 ${y_sign * track_separation/2} 0" rpy="0 0 0"/>
-    </joint>
-    <!-- FIX: Front and Rear slide laterally (mu=0.05), Mid has full grip (mu=1.0) -->
-    <xacro:agos_wheel side="${side}" y_sign="${y_sign}" pos="front" x="${wheel_x_offset}"  mu="0.05"/>
-    <xacro:agos_wheel side="${side}" y_sign="${y_sign}" pos="mid"   x="0"                  mu="1.0"/>
-    <xacro:agos_wheel side="${side}" y_sign="${y_sign}" pos="rear"  x="${-wheel_x_offset}" mu="0.05"/>
+    <!-- Outer road wheels slide sideways easily (mu 0.05) so the robot can
+         skid-steer; the two middle ones carry the grip (mu 1.0). -->
+    <xacro:agos_wheel side="${side}" y_sign="${y_sign}" pos="idler_front" x="0.29"    z="-0.05"       mu="0.8"/>
+    <xacro:agos_wheel side="${side}" y_sign="${y_sign}" pos="road_1"      x="0.2029"  z="${wheel_z}" mu="0.05"/>
+    <xacro:agos_wheel side="${side}" y_sign="${y_sign}" pos="road_2"      x="0.0759"  z="${wheel_z}" mu="1.0"/>
+    <xacro:agos_wheel side="${side}" y_sign="${y_sign}" pos="road_3"      x="-0.0511" z="${wheel_z}" mu="1.0"/>
+    <xacro:agos_wheel side="${side}" y_sign="${y_sign}" pos="road_4"      x="-0.2058" z="${wheel_z}" mu="0.05"/>
+    <xacro:agos_wheel side="${side}" y_sign="${y_sign}" pos="idler_rear"  x="-0.29"   z="-0.05"       mu="0.8"/>
   </xacro:macro>
-  <!-- Differential Drive Plugin -->
+  <!-- Differential Drive Plugin: every wheel on a side turns together, like a track -->
   <gazebo>
     <plugin filename="gz-sim-diff-drive-system" name="gz::sim::systems::DiffDrive">
-      <left_joint>left_wheel_front_joint</left_joint>
-      <left_joint>left_wheel_mid_joint</left_joint>
-      <left_joint>left_wheel_rear_joint</left_joint>
-      <right_joint>right_wheel_front_joint</right_joint>
-      <right_joint>right_wheel_mid_joint</right_joint>
-      <right_joint>right_wheel_rear_joint</right_joint>
+      <left_joint>left_wheel_idler_front_joint</left_joint>
+      <left_joint>left_wheel_road_1_joint</left_joint>
+      <left_joint>left_wheel_road_2_joint</left_joint>
+      <left_joint>left_wheel_road_3_joint</left_joint>
+      <left_joint>left_wheel_road_4_joint</left_joint>
+      <left_joint>left_wheel_idler_rear_joint</left_joint>
+      <right_joint>right_wheel_idler_front_joint</right_joint>
+      <right_joint>right_wheel_road_1_joint</right_joint>
+      <right_joint>right_wheel_road_2_joint</right_joint>
+      <right_joint>right_wheel_road_3_joint</right_joint>
+      <right_joint>right_wheel_road_4_joint</right_joint>
+      <right_joint>right_wheel_idler_rear_joint</right_joint>
       <wheel_separation>${track_separation}</wheel_separation>
-      <wheel_radius>${track_radius}</wheel_radius>
+      <wheel_radius>${wheel_radius}</wheel_radius>
       <topic>cmd_vel</topic>
       <odom_topic>odom</odom_topic>

File: practice_agos/agos_sim/urdf/agos_urdf.xacro (robot description, xacro)
@@ -2,32 +2,40 @@
 <robot name="agos" xmlns:xacro="http://www.ros.org/wiki/xacro">
   <!-- ===================== Dimensions =====================
-       Everything is derived from the working tracked_robot track:
-         track belt 0.6 long x 0.06 wide x 0.16 tall (radius 0.08)
-         track centre-to-centre separation 0.36  -> 0.30 gap between the tracks
-       Envelope: 600 x 420 x 320 mm (L x W x H), excluding LiDAR and pole.
-       Lower half = tracks, upper half = body. chassis_height = 4*track_radius. -->
-  <!-- Track (matches the working track code) -->
-  <xacro:property name="track_radius"     value="0.08"/>
-  <xacro:property name="track_width"      value="0.06"/>
-  <xacro:property name="track_separation" value="0.36"/>
-  <xacro:property name="track_length"     value="0.6"/>
-  <xacro:property name="wheel_mass"       value="0.5"/>
-  <xacro:property name="track_mu"         value="0.4"/>
-  <!-- Envelope (derived) -->
-  <xacro:property name="chassis_length" value="${track_length}"/>
-  <xacro:property name="chassis_width"  value="${track_separation + track_width}"/>
-  <xacro:property name="chassis_height" value="${4*track_radius}"/>
+       Measured from the CAD export Designs/STL/AGOS V1.stl (Fusion, mm).
+       The CAD model faces +y; here it is rotated so +x is forward, and scaled
+       to metres. base_link sits at the CAD origin, 0.178 m above the ground.
+         Body envelope : 0.711 L x 0.381 W x 0.476 H (ground to top of LiDAR)
+         Tracks        : 0.042 wide tread, centred 0.1436 m either side,
+                         flat contact patch from x = -0.21 to +0.21
+         Road wheels   : 4 rollers per side inside each track
+         Rear tether conduit (about 0.69 m long) is visual only.
+       The meshes in meshes/agos_*.stl are a simplified copy of that CAD file
+       (see tools/convert_robot_stl.py). -->
+  <!-- Track / wheels -->
+  <xacro:property name="ground_to_base"   value="0.178"/>   <!-- ground -> base_link -->
+  <xacro:property name="track_y"          value="0.1436"/>  <!-- track centre, either side -->
+  <xacro:property name="track_width"      value="0.042"/>
+  <xacro:property name="track_separation" value="${2*track_y}"/>
+  <xacro:property name="wheel_radius"     value="0.0385"/>
+  <xacro:property name="wheel_z"          value="${wheel_radius - ground_to_base}"/>
+  <xacro:property name="wheel_mass"       value="0.25"/>
+  <!-- Chassis -->
+  <xacro:property name="chassis_length" value="0.66"/>
+  <xacro:property name="chassis_width"  value="0.381"/>  <!-- overall, incl. tracks -->
+  <xacro:property name="chassis_height" value="0.40"/>
   <xacro:property name="chassis_mass"   value="15.0"/>
-  <xacro:property name="wheel_x_offset" value="${chassis_length/2 - track_radius}"/>
-  <!-- Belly pan between the tracks (z measured from the ground) -->
-  <xacro:property name="belly_height"   value="0.10"/>
-  <xacro:property name="belly_center_z" value="0.10"/>
-  <!-- Body above the tracks, measured from the track top -->
-  <xacro:property name="body_height"   value="${chassis_height/2}"/>
-  <xacro:property name="lidar_mount_h" value="0.05"/>
-  <xacro:property name="whip_length"   value="0.28"/>
   <xacro:include filename="$(find agos_sim)/urdf/agos_materials.xacro"/>
   <xacro:include filename="$(find agos_sim)/urdf/agos_tracks.xacro"/>
   <xacro:include filename="$(find agos_sim)/urdf/agos_sensors.xacro"/>
+  <!-- One coloured part of the CAD model (already in metres, +x forward) -->
+  <xacro:macro name="agos_mesh_visual" params="part material">
+    <visual>
+      <origin xyz="0 0 0" rpy="0 0 0"/>
+      <geometry>
+        <mesh filename="package://agos_sim/meshes/agos_${part}.stl"/>
+      </geometry>
+      <material name="${material}"/>
+    </visual>
+  </xacro:macro>
   <!-- ===================== base_footprint -> base_link -> chassis_link ===================== -->
   <link name="base_footprint"/>
@@ -35,76 +43,43 @@
     <parent link="base_footprint"/>
     <child link="base_link"/>
-    <origin xyz="0 0 ${track_radius}" rpy="0 0 0"/>
+    <origin xyz="0 0 ${ground_to_base}" rpy="0 0 0"/>
   </joint>
   <link name="base_link"/>
-  <!-- chassis_link origin = envelope center (ground + chassis_height/2 = track top) -->
   <joint name="base_link_to_chassis" type="fixed">
     <parent link="base_link"/>
     <child link="chassis_link"/>
-    <origin xyz="0 0 ${chassis_height/2 - track_radius}" rpy="0 0 0"/>
+    <origin xyz="0 0 0" rpy="0 0 0"/>
   </joint>
   <link name="chassis_link">
-    <!-- Green belly pan, between the tracks -->
-    <visual>
-      <origin xyz="0 0 ${belly_center_z - chassis_height/2}" rpy="0 0 0"/>
-      <geometry>
-        <box size="${chassis_length - 0.06} ${track_separation - track_width - 0.004} ${belly_height}"/>
-      </geometry>
-      <material name="agos_green_body"/>
-    </visual>
-    <!-- Silver main body enclosure -->
-    <visual>
-      <origin xyz="0 0 ${(body_height - 0.01)/2}" rpy="0 0 0"/>
-      <geometry>
-        <box size="${chassis_length - 0.08} ${chassis_width - 0.02} ${body_height - 0.01}"/>
-      </geometry>
-      <material name="agos_silver_enclosure"/>
-    </visual>
-    <!-- Green top lid plate -->
-    <visual>
-      <origin xyz="0 0 ${body_height - 0.005}" rpy="0 0 0"/>
-      <geometry>
-        <box size="${chassis_length - 0.10} ${chassis_width - 0.04} 0.01"/>
-      </geometry>
-      <material name="agos_green_body"/>
-    </visual>
-    <!-- Front roll-cage arch -->
-    <visual>
-      <origin xyz="0.17 0 ${body_height/2}" rpy="0 0 0"/>
-      <geometry>
-        <box size="0.03 ${chassis_width} ${body_height + 0.01}"/>
-      </geometry>
-      <material name="agos_dark_grey_frame"/>
-    </visual>
-    <!-- Rear roll-cage arch -->
-    <visual>
-      <origin xyz="-0.17 0 ${body_height/2}" rpy="0 0 0"/>
-      <geometry>
-        <box size="0.03 ${chassis_width} ${body_height + 0.01}"/>
-      </geometry>
-      <material name="agos_dark_grey_frame"/>
-    </visual>
-    <!-- Rear whip pole / antenna (visual only) -->
-    <visual>
-      <origin xyz="${-chassis_length/2 - whip_length/2 + 0.05} 0 ${body_height/2}" rpy="0 ${pi/2} 0"/>
-      <geometry>
-        <cylinder radius="0.01" length="${whip_length}"/>
-      </geometry>
-      <material name="agos_sensor_dark"/>
-    </visual>
-    <!-- Yellow LiDAR pedestal (the LiDAR itself is in agos_sensors.xacro) -->
-    <visual>
-      <origin xyz="0 0 ${body_height + lidar_mount_h/2}" rpy="0 0 0"/>
-      <geometry>
-        <box size="0.08 0.08 ${lidar_mount_h}"/>
-      </geometry>
-      <material name="agos_lidar_yellow"/>
-    </visual>
-    <!-- Collision: upper body only. Tracks/wheels carry ground contact. -->
+    <!-- Visual: the CAD model, split by its colours -->
+    <xacro:agos_mesh_visual part="body"    material="agos_body_grey"/>
+    <xacro:agos_mesh_visual part="treads"  material="agos_tread_red"/>
+    <xacro:agos_mesh_visual part="accents" material="agos_accent_yellow"/>
+    <xacro:agos_mesh_visual part="light"   material="agos_light_grey"/>
+    <xacro:agos_mesh_visual part="green"   material="agos_green_body"/>
+    <xacro:agos_mesh_visual part="dark"    material="agos_sensor_dark"/>
+    <!-- Collision: simple boxes that follow the body's cross-section (lid
+         0.28 m wide on top, narrowing to the belly between the tracks). The
+         tracks' ground contact is carried by the wheel cylinders in
+         agos_tracks.xacro. -->
+    <!-- Lid and upper hull -->
     <collision>
-      <origin xyz="0 0 ${body_height/2}" rpy="0 0 0"/>
-      <geometry>
-        <box size="${chassis_length - 0.08} ${chassis_width} ${body_height}"/>
-      </geometry>
+      <origin xyz="0 0 0.1543" rpy="0 0 0"/>
+      <geometry><box size="${chassis_length} 0.28 0.1486"/></geometry>
+    </collision>
+    <!-- Lower hull and belly between the tracks -->
+    <collision>
+      <origin xyz="0 0 -0.01" rpy="0 0 0"/>
+      <geometry><box size="0.62 0.22 0.18"/></geometry>
+    </collision>
+    <!-- Camera housing on the front of the lid -->
+    <collision>
+      <origin xyz="0.3066 0 0.2400" rpy="0 0 0"/>
+      <geometry><box size="0.099 0.165 0.074"/></geometry>
+    </collision>
+    <!-- LiDAR and its pedestal -->
+    <collision>
+      <origin xyz="0 0 0.2508" rpy="0 0 0"/>
+      <geometry><cylinder radius="0.04" length="0.0952"/></geometry>
     </collision>
     <inertial>
