Commit message: Improved Simulation Environment
- Upscaled Pipe w/ Textures
- New Map for Roaming
- Removed Solid Tether from AGOS model

File: practice_agos/agos_sim/urdf/agos_sensors.xacro (robot description, xacro)
@@ -129,6 +129,8 @@
       <origin xyz="0 0 0.01" rpy="0 0 0"/>
     </joint>
-    <!-- Requires the gz-sim-imu-system world plugin (in worlds/agos_pipe.sdf
-         and worlds/agos_world.sdf) or this topic stays silent. -->
+    <!-- Requires the gz-sim-imu-system world plugin (in all three worlds)
+         or this topic stays silent. The EKF (config/ekf.yaml) takes the
+         robot's turn rate from this gyro. The noise is roughly that of a
+         low-cost MEMS IMU. -->
     <gazebo reference="imu_link">
       <sensor name="agos_imu" type="imu">
@@ -137,4 +139,16 @@
         <topic>imu/data</topic>
         <gz_frame_id>imu_link</gz_frame_id>
+        <imu>
+          <angular_velocity>
+            <x><noise type="gaussian"><mean>0</mean><stddev>0.002</stddev></noise></x>
+            <y><noise type="gaussian"><mean>0</mean><stddev>0.002</stddev></noise></y>
+            <z><noise type="gaussian"><mean>0</mean><stddev>0.002</stddev></noise></z>
+          </angular_velocity>
+          <linear_acceleration>
+            <x><noise type="gaussian"><mean>0</mean><stddev>0.02</stddev></noise></x>
+            <y><noise type="gaussian"><mean>0</mean><stddev>0.02</stddev></noise></y>
+            <z><noise type="gaussian"><mean>0</mean><stddev>0.02</stddev></noise></z>
+          </linear_acceleration>
+        </imu>
       </sensor>
     </gazebo>

File: practice_agos/agos_sim/urdf/agos_tracks.xacro (robot description, xacro)
@@ -61,5 +61,5 @@
       <right_joint>right_wheel_road_4_joint</right_joint>
       <right_joint>right_wheel_idler_rear_joint</right_joint>
-      <wheel_separation>${track_separation}</wheel_separation>
+      <wheel_separation>${track_separation * skid_factor}</wheel_separation>
       <wheel_radius>${wheel_radius}</wheel_radius>
       <topic>cmd_vel</topic>

File: practice_agos/agos_sim/urdf/agos_urdf.xacro (robot description, xacro)
@@ -9,5 +9,6 @@
                          flat contact patch from x = -0.21 to +0.21
          Road wheels   : 4 rollers per side inside each track
-         Rear tether conduit (about 0.69 m long) is visual only.
+         The tether tube out of the back of the CAD model is left out of the
+         meshes (tools/convert_robot_stl.py): it is a cable, not a rigid part.
        The meshes in meshes/agos_*.stl are a simplified copy of that CAD file
        (see tools/convert_robot_stl.py). -->
@@ -17,4 +18,11 @@
   <xacro:property name="track_width"      value="0.042"/>
   <xacro:property name="track_separation" value="${2*track_y}"/>
+  <!-- A tracked robot skids sideways when it turns, so it turns less than
+       its track speeds say: in Gazebo it turns 0.77x as far as plain
+       diff-drive maths predicts. DiffDrive uses this wider "effective" track
+       separation (0.287 m / 0.77) so a commanded turn rate is what the robot
+       really does, and /odom reports the turn it really made. Re-measure if
+       you change the wheels or their friction. -->
+  <xacro:property name="skid_factor"      value="1.30"/>
   <xacro:property name="wheel_radius"     value="0.0385"/>
   <xacro:property name="wheel_z"          value="${wheel_radius - ground_to_base}"/>

File: practice_agos/build/agos_sim/urdf/agos_materials.xacro (robot description, xacro)
@@ -1 +1 @@
-/home/reuel/practice_agos/agos_sim/urdf/agos_materials.xacro
+/run/media/sazoverse/3228b30c-6f8e-4590-8359-973ebc8d68b0/School/Others/AGOS/Testing/ROS2/agos_gazebo_rviz_test/practice_agos/agos_sim/urdf/agos_materials.xacro

File: practice_agos/build/agos_sim/urdf/agos_sensors.xacro (robot description, xacro)
@@ -1 +1 @@
-/home/reuel/practice_agos/agos_sim/urdf/agos_sensors.xacro
+/run/media/sazoverse/3228b30c-6f8e-4590-8359-973ebc8d68b0/School/Others/AGOS/Testing/ROS2/agos_gazebo_rviz_test/practice_agos/agos_sim/urdf/agos_sensors.xacro

File: practice_agos/build/agos_sim/urdf/agos_tracks.xacro (robot description, xacro)
@@ -1 +1 @@
-/home/reuel/practice_agos/agos_sim/urdf/agos_tracks.xacro
+/run/media/sazoverse/3228b30c-6f8e-4590-8359-973ebc8d68b0/School/Others/AGOS/Testing/ROS2/agos_gazebo_rviz_test/practice_agos/agos_sim/urdf/agos_tracks.xacro

File: practice_agos/build/agos_sim/urdf/agos_urdf.xacro (robot description, xacro)
@@ -1 +1 @@
-/home/reuel/practice_agos/agos_sim/urdf/agos_urdf.xacro
+/run/media/sazoverse/3228b30c-6f8e-4590-8359-973ebc8d68b0/School/Others/AGOS/Testing/ROS2/agos_gazebo_rviz_test/practice_agos/agos_sim/urdf/agos_urdf.xacro

File: practice_agos/build/agos_sim/urdf/tracked_robot.urdf.xacro (robot description, xacro)
@@ -1 +1 @@
-/home/reuel/practice_agos/agos_sim/urdf/tracked_robot.urdf.xacro
+/run/media/sazoverse/3228b30c-6f8e-4590-8359-973ebc8d68b0/School/Others/AGOS/Testing/ROS2/agos_gazebo_rviz_test/practice_agos/agos_sim/urdf/tracked_robot.urdf.xacro

File: practice_agos/install/agos_sim/share/agos_sim/urdf/agos_materials.xacro (robot description, xacro)
@@ -1 +1 @@
-/home/reuel/practice_agos/build/agos_sim/urdf/agos_materials.xacro
+/run/media/sazoverse/3228b30c-6f8e-4590-8359-973ebc8d68b0/School/Others/AGOS/Testing/ROS2/agos_gazebo_rviz_test/practice_agos/build/agos_sim/urdf/agos_materials.xacro

File: practice_agos/install/agos_sim/share/agos_sim/urdf/agos_sensors.xacro (robot description, xacro)
@@ -1 +1 @@
-/home/reuel/practice_agos/build/agos_sim/urdf/agos_sensors.xacro
+/run/media/sazoverse/3228b30c-6f8e-4590-8359-973ebc8d68b0/School/Others/AGOS/Testing/ROS2/agos_gazebo_rviz_test/practice_agos/build/agos_sim/urdf/agos_sensors.xacro

File: practice_agos/install/agos_sim/share/agos_sim/urdf/agos_tracks.xacro (robot description, xacro)
@@ -1 +1 @@
-/home/reuel/practice_agos/build/agos_sim/urdf/agos_tracks.xacro
+/run/media/sazoverse/3228b30c-6f8e-4590-8359-973ebc8d68b0/School/Others/AGOS/Testing/ROS2/agos_gazebo_rviz_test/practice_agos/build/agos_sim/urdf/agos_tracks.xacro

File: practice_agos/install/agos_sim/share/agos_sim/urdf/agos_urdf.xacro (robot description, xacro)
@@ -1 +1 @@
-/home/reuel/practice_agos/build/agos_sim/urdf/agos_urdf.xacro
+/run/media/sazoverse/3228b30c-6f8e-4590-8359-973ebc8d68b0/School/Others/AGOS/Testing/ROS2/agos_gazebo_rviz_test/practice_agos/build/agos_sim/urdf/agos_urdf.xacro

File: practice_agos/install/agos_sim/share/agos_sim/urdf/tracked_robot.urdf.xacro (robot description, xacro)
@@ -1 +1 @@
-/home/reuel/practice_agos/build/agos_sim/urdf/tracked_robot.urdf.xacro
+/run/media/sazoverse/3228b30c-6f8e-4590-8359-973ebc8d68b0/School/Others/AGOS/Testing/ROS2/agos_gazebo_rviz_test/practice_agos/build/agos_sim/urdf/tracked_robot.urdf.xacro

Commit message: Full Exploration + Larger Map

File: practice_agos/agos_sim/urdf/agos_sensors.xacro (robot description, xacro)
@@ -138,6 +138,7 @@
     <!-- Requires the gz-sim-imu-system world plugin (in all three worlds)
          or this topic stays silent. The EKF (config/ekf.yaml) takes the
-         robot's turn rate from this gyro. The noise is roughly that of a
-         low-cost MEMS IMU. -->
+         robot's turn rate from this gyro, through imu_level (corrected for
+         the robot's tilt). The noise is roughly that of a low-cost MEMS
+         IMU. -->
     <gazebo reference="imu_link">
       <sensor name="agos_imu" type="imu">

File: practice_agos/agos_sim/urdf/agos_tracks.xacro (robot description, xacro)
@@ -7,5 +7,5 @@
          2 idler wheels : the raised front/rear ends of the track, so the
                           robot can climb onto lips, debris and pipe walls -->
-  <xacro:macro name="agos_wheel" params="side y_sign pos x z mu">
+  <xacro:macro name="agos_wheel" params="side y_sign pos x z mu mu_side">
     <link name="${side}_wheel_${pos}">
       <collision>
@@ -31,18 +31,24 @@
       <dynamics damping="0.1" friction="0.05"/>
     </joint>
+    <!-- mu1 acts along fdir1, the axle (sideways); mu2 along the track -->
     <gazebo reference="${side}_wheel_${pos}">
-      <mu1>${mu}</mu1>
+      <mu1>${mu_side}</mu1>
       <mu2>${mu}</mu2>
+      <fdir1>0 0 1</fdir1>
     </gazebo>
   </xacro:macro>
   <xacro:macro name="agos_track" params="side y_sign">
-    <!-- Outer road wheels slide sideways easily (mu 0.05) so the robot can
-         skid-steer; the two middle ones carry the grip (mu 1.0). -->
-    <xacro:agos_wheel side="${side}" y_sign="${y_sign}" pos="idler_front" x="0.29"    z="-0.05"       mu="0.8"/>
-    <xacro:agos_wheel side="${side}" y_sign="${y_sign}" pos="road_1"      x="0.2029"  z="${wheel_z}" mu="0.05"/>
-    <xacro:agos_wheel side="${side}" y_sign="${y_sign}" pos="road_2"      x="0.0759"  z="${wheel_z}" mu="1.0"/>
-    <xacro:agos_wheel side="${side}" y_sign="${y_sign}" pos="road_3"      x="-0.0511" z="${wheel_z}" mu="1.0"/>
-    <xacro:agos_wheel side="${side}" y_sign="${y_sign}" pos="road_4"      x="-0.2058" z="${wheel_z}" mu="0.05"/>
-    <xacro:agos_wheel side="${side}" y_sign="${y_sign}" pos="idler_rear"  x="-0.29"   z="-0.05"       mu="0.8"/>
+    <!-- Along the track every road wheel grips (mu 1.0), as a track does.
+         Sideways the outer road wheels slide easily (mu_side 0.05) so the
+         robot can skid-steer, and the two middle ones grip. When the outer
+         ones slid both ways, the robot stalled wherever the floor curved up
+         under a track (the benching beside a manhole opening): the middle
+         wheels lifted off the floor and the outer ones could not push. -->
+    <xacro:agos_wheel side="${side}" y_sign="${y_sign}" pos="idler_front" x="0.29"    z="-0.05"       mu="0.8" mu_side="0.8"/>
+    <xacro:agos_wheel side="${side}" y_sign="${y_sign}" pos="road_1"      x="0.2029"  z="${wheel_z}" mu="1.0" mu_side="0.05"/>
+    <xacro:agos_wheel side="${side}" y_sign="${y_sign}" pos="road_2"      x="0.0759"  z="${wheel_z}" mu="1.0" mu_side="1.0"/>
+    <xacro:agos_wheel side="${side}" y_sign="${y_sign}" pos="road_3"      x="-0.0511" z="${wheel_z}" mu="1.0" mu_side="1.0"/>
+    <xacro:agos_wheel side="${side}" y_sign="${y_sign}" pos="road_4"      x="-0.2058" z="${wheel_z}" mu="1.0" mu_side="0.05"/>
+    <xacro:agos_wheel side="${side}" y_sign="${y_sign}" pos="idler_rear"  x="-0.29"   z="-0.05"       mu="0.8" mu_side="0.8"/>
   </xacro:macro>
   <!-- Differential Drive Plugin: every wheel on a side turns together, like a track -->

File: practice_agos/agos_sim/urdf/agos_urdf.xacro (robot description, xacro)
@@ -24,11 +24,14 @@
   <xacro:property name="track_width"      value="0.042"/>
   <xacro:property name="track_separation" value="${2*track_y}"/>
-  <!-- A tracked robot skids sideways when it turns, so it turns less than
-       its track speeds say: in Gazebo it turns 0.77x as far as plain
-       diff-drive maths predicts. DiffDrive uses this wider "effective" track
-       separation (0.287 m / 0.77) so a commanded turn rate is what the robot
-       really does, and /odom reports the turn it really made. Re-measure if
-       you change the wheels or their friction. -->
-  <xacro:property name="skid_factor"      value="1.30"/>
+  <!-- DiffDrive uses track_separation x skid_factor as its wheel separation.
+       A tracked robot that skids when it turns needs more than 1: it turns
+       less than its track speeds say. This one turns 0.98-1.0x as far as
+       plain diff-drive maths predicts in Gazebo, because its outer road
+       wheels slide sideways (agos_tracks.xacro), so 1.0 makes a commanded
+       turn rate what the robot really does. (It was 1.30 when the outer
+       wheels had no grip along the track either.) If you change the wheels
+       or their friction, command a turn in place, compare with the turn
+       Gazebo reports, and set this to commanded / measured x this value. -->
+  <xacro:property name="skid_factor"      value="1.0"/>
   <xacro:property name="wheel_radius"     value="0.0385"/>
   <xacro:property name="wheel_z"          value="${wheel_radius - ground_to_base}"/>
